File: Electronics/macro_board_circuit/macro_board_circuit.kicad_sch (KiCad schematic)
At the start: 0 parts

Commit message: First circuit design
Only controller + switches/diodes so far
Parts:
- added D1, D2, D3, D4, D5, D6, D7, D8, D9: ~, Diode_THT:D_DO-35_SOD27_P7.62mm_Horizontal, symbol ScottoKeebs:Placeholder_Diode
- added S1, S2, S3, S4, S5, S6, S7, S8, S9: ~, ScottoKeebs_MX:MX_PCB_1.00u, symbol ScottoKeebs:Placeholder_Keyswitch
- added U1: nice_nano, Nice Nano:nice_nano, symbol Nice Nano:nice_nano
Connections:
- new net: D5.2 (A), S5.2
- new net: D8.2 (A), S8.2
- new net: D7.2 (A), S7.2
- new net: D1.2 (A), S1.2
- new net: D6.2 (A), S6.2
- new net: D2.2 (A), S2.2
- new net: D3.2 (A), S3.2
- new net: D9.2 (A), S9.2
- new net: D4.2 (A), S4.2
- new net Col 0: S1.1, S4.1, S7.1, U1.10 (P0.11)
- new net Col 1: S2.1, S5.1, S8.1, U1.11 (P1.04)
- new net Col 2: S3.1, S6.1, S9.1, U1.12 (P1.06)
- new net Row 0: D1.1 (K), D2.1 (K), D3.1 (K), U1.5 (P0.17)
- new net Row 1: D4.1 (K), D5.1 (K), D6.1 (K), U1.6 (P0.20)
- new net Row 2: D7.1 (K), D8.1 (K), D9.1 (K), U1.7 (P0.22)

Commit message: Added EC11 + fill volume
Added the EC11 encoder/switch and a copper fill volume to the PCB.
Parts:
- added R1: 10k, Resistor_THT:R_Axial_DIN0207_L6.3mm_D2.5mm_P10.16mm_Horizontal, symbol ScottoKeebs:Placeholder_Resistor
- added SW1: RotaryEncoder_Switch_MP, Rotary_Encoder:RotaryEncoder_Alps_EC11E-Switch_Vertical_H20mm, symbol Device:RotaryEncoder_Switch_MP
Connections:
- net Switch Pin: now reaches U1.17 (P1.15)
- net Switch Pin: now also R1.1, SW1.S1
- net VCC Pin: now reaches U1.21 (VCC)
- net VCC Pin: now also SW1.S2
- net GND Pin: now reaches U1.23 (GND)
- net GND Pin: now also R1.2, SW1.C
- net EC - A: now reaches U1.8 (P0.24)
- net EC - A: now also SW1.A
- net EC - B: now reaches U1.9 (P1.00)
- net EC - B: now also SW1.B
